Commit message: reduced inflation radious + increased rocker tension to improve movement

File: urdf/macros.xacro (robot description, xacro)
@@ -227,5 +227,6 @@
       <child link="${link_prefix}rocker_L_link"/>
       <axis xyz="0 1 0"/>
-      <limit effort="100.0" lower="-0.24" upper="0.24" velocity="100.0"/>
+      <!-- <limit effort="100.0" lower="-0.24" upper="0.24" velocity="100.0"/> -->
+      <limit effort="1000.0" lower="-0.05" upper="0.05" velocity="0.1"/>
       <dynamics friction="1.0" damping="0.1"/>
     </joint>
@@ -235,5 +236,6 @@
       <child link="${link_prefix}rocker_R_link"/>
       <axis xyz="0 1 0"/>
-      <limit effort="100.0" lower="-0.24" upper="0.24" velocity="100.0"/>
+      <!-- <limit effort="100.0" lower="-0.24" upper="0.24" velocity="100.0"/> -->
+      <limit effort="1000.0" lower="-0.05" upper="0.05" velocity="0.1"/>
       <dynamics friction="1.0" damping="0.1"/>
       <mimic joint="rocker_L_joint"/>
@@ -446,5 +448,5 @@
         <jointA>rocker_L_joint</jointA>
         <jointB>rocker_R_joint</jointB>
-        <forceConstant>100.0</forceConstant>
+        <forceConstant>10.0</forceConstant>
       </plugin>
     </gazebo>
@@ -479,5 +481,5 @@
 	        <wheelDiameter>1</wheelDiameter>
           <broadcastTF>1</broadcastTF> -->
-          <wheelTorque>1000</wheelTorque>
+          <wheelTorque>10000</wheelTorque>
           <!-- <wheelAcceleration>1.8</wheelAcceleration> -->
           <!-- <commandTopic>$(arg robot_ns)/cmd_vel</commandTopic> -->

Commit message: removed wall, recoloured others and added pc box

File: urdf/macros.xacro (robot description, xacro)
@@ -205,4 +205,15 @@
       <material>Gazebo/Black</material>
   </gazebo>
+  <link name="${link_prefix}box">
+    <visual>
+      <origin xyz="-0.1 0 0" rpy="0 0 0"/>
+      <geometry>
+        <box size="0.15 0.2 0.1"/>
+      </geometry>
+      <material name="white">
+        <color rgba="1 1 1 1"/>
+    </material>
+    </visual>
+  </link>
     <link name="${link_prefix}camera_frame"/>
     <link name="${link_prefix}camera_optical_frame"/>
@@ -326,4 +337,10 @@
       <parent link="${link_prefix}base_link"/>
       <child link="${link_prefix}laser"/>
+  </joint>
+  <!-- Attach the box to the base footprint with a fixed joint -->
+  <joint name="box_joint" type="fixed">
+    <parent link="$(arg robot_ns)/base_link"/>
+    <child link="${link_prefix}box"/>
+    <origin xyz="0 0 0.05" rpy="0 0 0"/> <!-- Adjust the z value to half the height of the box -->
   </joint>
   </xacro:macro>
